File: pcb/timed_off.sch (KiCad schematic (older format))
At the start: 19 parts, among them J1 L, J2 N, J3 L, J4 N, U1 ATtiny10-TS, U2 SPA4191

Commit message: add footprints
Parts:
- C1: value 0.33uF -> 0.47uF; footprint (none) -> Capacitor_THT:C_Rect_L29.0mm_W11.0mm_P27.50mm_MKT
- C2: footprint (none) -> Capacitor_THT:CP_Radial_D8.0mm_P3.80mm
- C3: footprint (none) -> Capacitor_THT:C_Disc_D6.0mm_W2.5mm_P5.00mm
- D2: value 5.1V -> 4.7V; footprint (none) -> Diode_THT:D_DO-35_SOD27_P7.62mm_Horizontal
- F1: value Fuse -> 2A; footprint (none) -> Resistor_THT:R_Axial_DIN0309_L9.0mm_D3.2mm_P5.08mm_Vertical
- R1: value 1M -> 820k; footprint (none) -> Resistor_THT:R_Axial_DIN0207_L6.3mm_D2.5mm_P10.16mm_Horizontal
- R2: footprint (none) -> Resistor_THT:R_Axial_DIN0411_L9.9mm_D3.6mm_P7.62mm_Vertical
- R3, R5: value R -> 1.2k; footprint (none) -> Resistor_THT:R_Axial_DIN0207_L6.3mm_D2.5mm_P10.16mm_Horizontal
- R4: value R -> 560; footprint (none) -> Resistor_THT:R_Axial_DIN0207_L6.3mm_D2.5mm_P10.16mm_Horizontal
- R6: value 470 -> 220; footprint (none) -> Resistor_THT:R_Axial_DIN0207_L6.3mm_D2.5mm_P10.16mm_Horizontal
- U2: footprint (none) -> pl_SSR:SPA4191
Other:
- note added: "16mA"
- note added: "275V X2"
- note added: "4mA"
- note added: "Carbon Composite"
- note added: "Max Current: 29mA"
- note added: "Xc = 1/(2*pi*f*C1)\nXc = 1/(2*3.14*60Hz*0.47e-6F)\nXc = 5644ohms\n\nZc = |Xc|\nZall = sqrt(Zc^2 + R2^2)\n\nImax = (120Vrms * sqrt(2)) / Zall\nImax = 29mA"
- note removed: "10-35mA"
- moved on the sheet: D3, R4
Changed lines of the file:
@@
 P 2900 2500
 F 0 "F1" V 2980 2500 50  0000 C CNN
-F 1 "Fuse" V 2825 2500 50  0000 C CNN
-F 2 "" V 2830 2500 50  0001 C CNN
+F 1 "2A" V 2825 2500 50  0000 C CNN
+F 2 "Resistor_THT:R_Axial_DIN0309_L9.0mm_D3.2mm_P5.08mm_Vertical" V 2830 2500 50  0001 C CNN
 F 3 "~" H 2900 2500 50  0001 C CNN
 	1    2900 2500
@@
 P 3700 2500
 F 0 "C1" V 3550 2500 50  0000 C CNN
-F 1 "0.33uF" V 3850 2500 50  0000 C CNN
-F 2 "" H 3738 2350 50  0001 C CNN
+F 1 "0.47uF" V 3850 2500 50  0000 C CNN
+F 2 "Capacitor_THT:C_Rect_L29.0mm_W11.0mm_P27.50mm_MKT" H 3738 2350 50  0001 C CNN
 F 3 "~" H 3700 2500 50  0001 C CNN
 	1    3700 2500
@@
 P 3700 2200
 F 0 "R1" V 3780 2200 50  0000 C CNN
-F 1 "1M" V 3700 2200 50  0000 C CNN
-F 2 "" V 3630 2200 50  0001 C CNN
+F 1 "820k" V 3700 2200 50  0000 C CNN
+F 2 "Resistor_THT:R_Axial_DIN0207_L6.3mm_D2.5mm_P10.16mm_Horizontal" V 3630 2200 50  0001 C CNN
 F 3 "~" H 3700 2200 50  0001 C CNN
 	1    3700 2200
@@
 F 0 "R2" V 3780 3200 50  0000 C CNN
 F 1 "1k" V 3700 3200 50  0000 C CNN
-F 2 "" V 3630 3200 50  0001 C CNN
+F 2 "Resistor_THT:R_Axial_DIN0411_L9.9mm_D3.6mm_P7.62mm_Vertical" V 3630 3200 50  0001 C CNN
 F 3 "~" H 3700 3200 50  0001 C CNN
 	1    3700 3200
@@
 P 4900 3200
 F 0 "D2" H 4900 3300 50  0000 C CNN
-F 1 "5.1V" H 4900 3100 50  0000 C CNN
-F 2 "" H 4900 3200 50  0001 C CNN
+F 1 "4.7V" H 4900 3100 50  0000 C CNN
+F 2 "Diode_THT:D_DO-35_SOD27_P7.62mm_Horizontal" H 4900 3200 50  0001 C CNN
 F 3 "~" H 4900 3200 50  0001 C CNN
 	1    4900 3200
@@
 F 0 "C2" H 5225 3300 50  0000 L CNN
 F 1 "470uF" H 5225 3100 50  0000 L CNN
-F 2 "" H 5238 3050 50  0001 C CNN
+F 2 "Capacitor_THT:CP_Radial_D8.0mm_P3.80mm" H 5238 3050 50  0001 C CNN
 F 3 "~" H 5200 3200 50  0001 C CNN
 	1    5200 3200
@@
 F 0 "C3" V 6200 2850 50  0000 C CNN
 F 1 "100n" V 6500 2850 50  0000 C CNN
-F 2 "" H 6388 2700 50  0001 C CNN
+F 2 "Capacitor_THT:C_Disc_D6.0mm_W2.5mm_P5.00mm" H 6388 2700 50  0001 C CNN
 F 3 "~" H 6350 2850 50  0001 C CNN
 	1    6350 2850
@@
 P 7150 3450
 F 0 "R6" V 7230 3450 50  0000 C CNN
-F 1 "470" V 7150 3450 50  0000 C CNN
-F 2 "" V 7080 3450 50  0001 C CNN
+F 1 "220" V 7150 3450 50  0000 C CNN
+F 2 "Resistor_THT:R_Axial_DIN0207_L6.3mm_D2.5mm_P10.16mm_Horizontal" V 7080 3450 50  0001 C CNN
 F 3 "~" H 7150 3450 50  0001 C CNN
 	1    7150 3450
@@
 F 0 "U2" H 7750 3750 50  0000 L CNN
 F 1 "SPA4191" H 7950 3750 50  0000 L CNN
-F 2 "" H 7750 3350 50  0001 L CIN
+F 2 "pl_SSR:SPA4191" H 7750 3350 50  0001 L CIN
 F 3 "" H 7950 3550 50  0001 L CNN
 	1    7950 3550
@@
 Wire Wire Line
 	7550 3650 7550 3750
-Text Notes 7350 3550 0    50   ~ 0
-10-35mA
+Text Notes 7350 3450 0    50   ~ 0
+16mA
 Text Label 3200 2500 0    50   ~ 0
 L
@@
 L Device:R R4
 U 1 1 60F0ACE3
-P 6850 3050
-F 0 "R4" V 6930 3050 50  0000 C CNN
-F 1 "R" V 6850 3050 50  0000 C CNN
-F 2 "" V 6780 3050 50  0001 C CNN
-F 3 "~" H 6850 3050 50  0001 C CNN
-	1    6850 3050
-	-1   0    0    1
+P 7150 2950
+F 0 "R4" V 7230 2950 50  0000 C CNN
+F 1 "560" V 7150 2950 50  0000 C CNN
+F 2 "Resistor_THT:R_Axial_DIN0207_L6.3mm_D2.5mm_P10.16mm_Horizontal" V 7080 2950 50  0001 C CNN
+F 3 "~" H 7150 2950 50  0001 C CNN
+	1    7150 2950
+	0    -1   -1   0
 $EndComp
 $Comp
 L Device:LED D3
 U 1 1 60F108C8
-P 7100 2800
-F 0 "D3" H 7100 2900 50  0000 C CNN
-F 1 "RED" H 7100 2700 50  0000 C CNN
-F 2 "LED_THT:LED_D5.0mm" H 7100 2800 50  0001 C CNN
-F 3 "~" H 7100 2800 50  0001 C CNN
-	1    7100 2800
+P 7850 2950
+F 0 "D3" H 7850 3050 50  0000 C CNN
+F 1 "RED" H 7850 2850 50  0000 C CNN
+F 2 "LED_THT:LED_D5.0mm" H 7850 2950 50  0001 C CNN
+F 3 "~" H 7850 2950 50  0001 C CNN
+	1    7850 2950
 	-1   0    0    1
 $EndComp
@@
 L power:GND #PWR08
 U 1 1 60F112C4
-P 7350 2900
-F 0 "#PWR08" H 7350 2650 50  0001 C CNN
-F 1 "GND" H 7350 2750 50  0000 C CNN
-F 2 "" H 7350 2900 50  0001 C CNN
-F 3 "" H 7350 2900 50  0001 C CNN
-	1    7350 2900
+P 8100 3050
+F 0 "#PWR08" H 8100 2800 50  0001 C CNN
+F 1 "GND" H 8100 2900 50  0000 C CNN
+F 2 "" H 8100 3050 50  0001 C CNN
+F 3 "" H 8100 3050 50  0001 C CNN
+	1    8100 3050
 	1    0    0    -1
 $EndComp
@@
 	6700 3350 6850 3350
 Wire Wire Line
-	6850 3350 6850 3200
-Wire Wire Line
-	6850 2900 6850 2800
-Wire Wire Line
-	6850 2800 6950 2800
-Wire Wire Line
-	7250 2800 7350 2800
-Wire Wire Line
-	7350 2800 7350 2900
-Text Notes 5800 4800 0    50   ~ 0
+	6850 3350 6850 2950
+Wire Wire Line
+	8000 2950 8100 2950
+Wire Wire Line
+	8100 2950 8100 3050
+Text Notes 5800 4900 0    50   ~ 0
 PB2
-Text Notes 6000 4800 0    50   ~ 0
+Text Notes 6000 4900 0    50   ~ 0
 PB3
-Text Notes 6200 4800 0    50   ~ 0
+Text Notes 6200 4900 0    50   ~ 0
 T
-Text Notes 5800 4900 0    50   ~ 0
-H
-Text Notes 6000 4900 0    50   ~ 0
-H
-Text Notes 6200 4900 0    50   ~ 0
-30min
 Text Notes 5800 5000 0    50   ~ 0
 H
 Text Notes 6000 5000 0    50   ~ 0
+H
+Text Notes 6200 5000 0    50   ~ 0
+30min
+Text Notes 5800 5100 0    50   ~ 0
+H
+Text Notes 6000 5100 0    50   ~ 0
 L
-Text Notes 6200 5000 0    50   ~ 0
+Text Notes 6200 5100 0    50   ~ 0
 3hrs
-Text Notes 5800 5100 0    50   ~ 0
-L
-Text Notes 6000 5100 0    50   ~ 0
-H
-Text Notes 6200 5100 0    50   ~ 0
-1hr
 Text Notes 5800 5200 0    50   ~ 0
 L
 Text Notes 6000 5200 0    50   ~ 0
+H
+Text Notes 6200 5200 0    50   ~ 0
+1hr
+Text Notes 5800 5300 0    50   ~ 0
 L
-Text Notes 6200 5200 0    50   ~ 0
+Text Notes 6000 5300 0    50   ~ 0
+L
+Text Notes 6200 5300 0    50   ~ 0
 x
 Wire Notes Line style solid
-	5800 5200 6450 5200
-Wire Notes Line style solid
-	6450 4700 5800 4700
-Wire Notes Line style solid
-	5800 4800 6450 4800
+	5800 5300 6450 5300
+Wire Notes Line style solid
+	6450 4800 5800 4800
+Wire Notes Line style solid
+	5800 4900 6450 4900
 Wire Notes Line
-	6000 4700 6000 5200
+	6000 4800 6000 5300
 Wire Notes Line
-	6200 4700 6200 5200
+	6200 4800 6200 5300
 $Comp
 L Device:R R3
@@
 P 6800 4100
 F 0 "R3" V 6880 4100 50  0000 C CNN
-F 1 "R" V 6800 4100 50  0000 C CNN
-F 2 "" V 6730 4100 50  0001 C CNN
+F 1 "1.2k" V 6800 4100 50  0000 C CNN
+F 2 "Resistor_THT:R_Axial_DIN0207_L6.3mm_D2.5mm_P10.16mm_Horizontal" V 6730 4100 50  0001 C CNN
 F 3 "~" H 6800 4100 50  0001 C CNN
 	1    6800 4100
@@
 P 7000 4100
 F 0 "R5" V 7080 4100 50  0000 C CNN
-F 1 "R" V 7000 4100 50  0000 C CNN
-F 2 "" V 6930 4100 50  0001 C CNN
+F 1 "1.2k" V 7000 4100 50  0000 C CNN
+F 2 "Resistor_THT:R_Axial_DIN0207_L6.3mm_D2.5mm_P10.16mm_Horizontal" V 6930 4100 50  0001 C CNN
 F 3 "~" H 7000 4100 50  0001 C CNN
 	1    7000 4100
@@
 Wire Wire Line
 	7000 4300 7000 4250
-Text Notes 5800 4700 0    50   ~ 0
+Text Notes 5800 4800 0    50   ~ 0
 Timeout Settings
 Wire Notes Line style solid
-	6450 4600 5800 4600
-Wire Notes Line style solid
-	5800 4600 5800 5200
-Wire Notes Line style solid
-	6450 4600 6450 5200
+	6450 4700 5800 4700
+Wire Notes Line style solid
+	5800 4700 5800 5300
+Wire Notes Line style solid
+	6450 4700 6450 5300
 $Comp
 L Connector_Generic:Conn_01x01 J4
@@
 	3350 4550 8400 4550
 $Comp
-L power:PWR_FLAG #FLG0101
-U 1 1 60FC2601
-P 5200 2800
-F 0 "#FLG0101" H 5200 2875 50  0001 C CNN
-F 1 "PWR_FLAG" H 5200 2950 50  0000 C CNN
-F 2 "" H 5200 2800 50  0001 C CNN
-F 3 "~" H 5200 2800 50  0001 C CNN
-	1    5200 2800
-	1    0    0    -1
-$EndComp
-Wire Wire Line
-	5200 2800 5200 2850
-$Comp
-L power:PWR_FLAG #FLG0102
-U 1 1 60FC3BC6
-P 4050 2800
-F 0 "#FLG0102" H 4050 2875 50  0001 C CNN
-F 1 "PWR_FLAG" H 4050 2950 50  0000 C CNN
-F 2 "" H 4050 2800 50  0001 C CNN
-F 3 "~" H 4050 2800 50  0001 C CNN
-	1    4050 2800
-	1    0    0    -1
-$EndComp
-Wire Wire Line
-	4050 2800 4050 2850
-Connection ~ 4050 2850
-$Comp
 L Diode_Bridge:MB2S D1
 U 1 1 60FC8224
@@
 	1    0    0    -1
 $EndComp
+Text Notes 3550 2750 0    50   ~ 0
+275V X2
+Text Notes 3350 3400 0    50   ~ 0
+Carbon Composite
+Text Notes 4900 2800 0    50   ~ 0
+Max Current: 29mA
+Text Notes 3350 5400 0    50   ~ 0
+Xc = 1/(2*pi*f*C1)\nXc = 1/(2*3.14*60Hz*0.47e-6F)\nXc = 5644ohms\n\nZc = |Xc|\nZall = sqrt(Zc^2 + R2^2)\n\nImax = (120Vrms * sqrt(2)) / Zall\nImax = 29mA
+Wire Wire Line
+	6850 2950 7000 2950
+Wire Wire Line
+	7300 2950 7700 2950
+Text Notes 7350 2950 0    50   ~ 0
+4mA
 $EndSCHEMATC

Commit message: update
Other:
- note added: "2hrs"
- note removed: "x"
Changed lines of the file:
@@
 Text Notes 6200 4900 0    50   ~ 0
 T
-Text Notes 5800 5000 0    50   ~ 0
+Text Notes 5800 5300 0    50   ~ 0
 H
-Text Notes 6000 5000 0    50   ~ 0
+Text Notes 6000 5300 0    50   ~ 0
 H
 Text Notes 6200 5000 0    50   ~ 0
@@
 L
 Text Notes 6200 5100 0    50   ~ 0
-3hrs
+1hr
 Text Notes 5800 5200 0    50   ~ 0
 L
@@
 H
 Text Notes 6200 5200 0    50   ~ 0
-1hr
-Text Notes 5800 5300 0    50   ~ 0
+2hrs
+Text Notes 5800 5000 0    50   ~ 0
 L
-Text Notes 6000 5300 0    50   ~ 0
+Text Notes 6000 5000 0    50   ~ 0
 L
 Text Notes 6200 5300 0    50   ~ 0
-x
+3hrs
 Wire Notes Line style solid
 	5800 5300 6450 5300

Commit message: fix bridge footprint, add second dropper cap footprint
Parts:
- D1: footprint Diode_THT:Diode_Bridge_DIP-4_W7.62mm_P5.08mm -> pl_Rectifier:S1WB
Changed lines of the file:
@@
 F 0 "D1" H 4500 3125 50  0000 L CNN
 F 1 "S1WB" H 4500 3050 50  0000 L CNN
-F 2 "Diode_THT:Diode_Bridge_DIP-4_W7.62mm_P5.08mm" H 4550 2975 50  0001 L CNN
+F 2 "pl_Rectifier:S1WB" H 4550 2975 50  0001 L CNN
 F 3 "" H 4400 2850 50  0001 C CNN
 	1    4400 2850
